File: ExOneMicrorocessor/ExOneMicrorocessor.kicad_pcb (KiCad board)
At the start: 2 copper layers, 41 parts, among them IC1 STM32G041C8T6, IC2 FT230XS, J1 UJ2-MBH-3-SMT, J2 Conn_01x02, J3 02x03 Header, J4 01x03, J5 01x08, J6 01x10, J7 01x12, SW1 SW4Push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

Commit message: started PCB LAyout
Parts:
- removed J6: 01x10, Connector_PinHeader_2.54mm:PinHeader_1x10_P2.54mm_Vertical
- removed J7: 01x12, Connector_PinHeader_2.54mm:PinHeader_1x12_P2.54mm_Vertical
- C7, C8, Y2: moved to B.Cu
- J4: value 01x03 -> Conn_01x17; footprint Connector_PinHeader_2.54mm:PinHeader_1x03_P2.54mm_Vertical -> Connector_PinHeader_2.54mm:PinHeader_1x17_P2.54mm_Vertical; moved to B.Cu
- J5: value 01x08 -> Conn_01x17; footprint Connector_PinHeader_2.54mm:PinHeader_1x08_P2.54mm_Vertical -> Connector_PinHeader_2.54mm:PinHeader_1x17_P2.54mm_Vertical; moved to B.Cu
- SW1: value SW4Push -> SW_Push; footprint Button_Switch_THT:SW_PUSH_6mm -> ExOneFootprints:PTS636SM25SMTRLFS
- moved J2 102.1 mm to (160.2, 67.6), turned to 0 degrees
- moved D1 88.9 mm to (161.4, 71.5)
- moved R7 88.3 mm to (161.9, 90.8), turned to 0 degrees
- moved F1 85.2 mm to (163.0, 75.3), turned to 90 degrees
- moved U1 82.9 mm to (161.7, 84.1), turned to 270 degrees
- moved Y2 80.7 mm to (156.5, 99.9), turned to 180 degrees
- moved C17 78.3 mm to (160.2, 89.0), turned to 0 degrees
- moved C6 77.7 mm to (160.6, 100.7), turned to 270 degrees
- moved C19 77.0 mm to (160.2, 94.2), turned to 0 degrees
- moved C16 76.6 mm to (162.1, 78.6)
- moved C18 76.5 mm to (160.2, 92.6)
- moved C5 73.7 mm to (163.1, 100.7), turned to 270 degrees
- moved C7 72.1 mm to (162.4, 95.5), turned to 270 degrees
- moved R3 69.1 mm to (160.4, 122.4), turned to 0 degrees
- moved R6 67.8 mm to (156.7, 102.1)
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Connections:
- net VCCIO renamed 3VLn
- J4 pad 2: PA0 -> PB9
- J4 pad 3: PA1 -> PB8
- J5 pad 1: PA4 -> PA0
- J5 pad 2: PA5 -> Net-(J5-Pad2)
- J5 pad 3: PA7 -> PA4
- J5 pad 4: PB0 -> PA5
- J5 pad 5: PB2 -> PA7
- J5 pad 6: PB10 -> PB0
- J5 pad 7: PB11 -> PB2
- J5 pad 8: PB12 -> PB10
- R5 pad 2: +3.3VA -> +3V3
- SW1 pad 1: GND -> Net-(R5-Pad1)
- SW1 pad 2: Net-(R5-Pad1) -> GND
Routing:
- net +3V3: track 0.00 -> 83.6 mm, vias 0 -> 2
- net GND: track 0.00 -> 63.8 mm, vias 0 -> 22
- net RTS: track 0.00 -> 36.8 mm, vias 0 -> 2
- net CTS: track 0.00 -> 35.7 mm, vias 0 -> 2
- net +5V: track 0.00 -> 35.7 mm
- net PA0: track 0.00 -> 35.2 mm, vias 0 -> 1
- net PA1: track 0.00 -> 33.8 mm, vias 0 -> 1
- net PA4: track 0.00 -> 31.8 mm, vias 0 -> 1
- net TX: track 0.00 -> 31.7 mm, vias 0 -> 2
- net PA5: track 0.00 -> 30.9 mm, vias 0 -> 1
- net PA7: track 0.00 -> 30.0 mm, vias 0 -> 1
- net RX: track 0.00 -> 29.3 mm, vias 0 -> 2
- net PC13: track 0.00 -> 28.8 mm
- net PB0: track 0.00 -> 26.6 mm, vias 0 -> 2
- net PB9: track 0.00 -> 26.3 mm
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- added copper zone on B.Cu, net GND
Other:
- board outline added: 33.5 x 62.7 mm

Commit message: FInished work on pcb , added some pads for 3v3 and gnd
Parts:
- added J6: Conn_01x02, Connector_PinHeader_2.54mm:PinHeader_1x02_P2.54mm_Vertical, F.Cu at (146.7, 124.9)
Connections:
- J5 pad 2: Net-(J5-Pad2) -> GND
Routing:
- net +3V3: track 83.6 -> 86.8 mm
- net TX: track 31.7 -> 33.7 mm
- net RTS: track 36.8 -> 37.4 mm
- added copper zone on F.Cu, net GND
