File: ExOneMicrorocessor/ExOneMicrorocessor.kicad_pcb (KiCad board)
At the start: 2 copper layers, 33.5 x 62.7 mm, 40 parts, among them IC1 STM32G041C8T6, IC2 FT230XS, J1 UJ2-MBH-3-SMT, J2 Conn_01x02, J3 02x03 Header, J4 Conn_01x17, J5 Conn_01x17, J6 Conn_01x02, SW1 SW_Push, U1 TPS77733DR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

Commit message: push for T
Parts:
- moved R4 0.09 mm to (149.6, 122.3)
Routing:
- net OSC_OUT: track 15.9 -> 19.8 mm
- net RTS: track 37.4 -> 33.9 mm
- net RX: track 29.6 -> 26.8 mm
- net CTS: track 35.7 -> 33.3 mm
- net +3V3: track 86.8 -> 85.5 mm
- net TX: track 33.7 -> 32.5 mm
- net PA7: track 30.0 -> 28.9 mm
- net PA15: track 6.35 -> 7.37 mm
- net PB2: track 25.6 -> 24.7 mm
- net PD1: track 9.78 -> 10.6 mm, vias 0 -> 1
- net PA5: track 30.9 -> 30.2 mm
- net PB10: track 23.7 -> 22.9 mm
- net PB4: track 17.3 -> 17.1 mm, vias 1 -> 0
Other:
- board text added: "3V3"
- board text added: "GND"
- board text added: "PA1"
- board text added: "PA10"
- board text added: "PA11"
- board text added: "PA12"
- board text added: "PA15"
- board text added: "PA4"
- board text added: "PA5"
- board text added: "PA7"
- board text added: "PA8"
- board text added: "PA9"
- board text added: "PB0"
- board text added: "PB10"
- board text added: "PB11"
- board text added: "PB12"
- board text added: "PB13"
- board text added: "PB14"
- board text added: "PB15"
- board text added: "PB2"
- board text added: "PB3"
- board text added: "PB4"
- board text added: "PB5"
- board text added: "PB6"
- board text added: "PB7"
- board text added: "PB8"
- board text added: "PB9"
- board text added: "PC13"
- board text added: "PC6"
- board text added: "PC7"
- board text added: "PD0"
- board text added: "PD1"
- board text added: "PD2"
- board text added: "PD3"
