File: ExOneMicrorocessor/ExOneMicrorocessor.sch (KiCad schematic (older format))
At the start: 41 parts, among them IC1 STM32G041C8T6, IC2 FT230XS, J1 UJ2-MBH-3-SMT, J2 Conn_01x02, J3 02x03 Header, J4 01x03, J5 01x08, J6 01x10, J7 01x12, SW1 SW4Push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

Commit message: started PCB LAyout
Parts:
- removed J4: 01x03, Connector_PinHeader_2.54mm:PinHeader_1x03_P2.54mm_Vertical, symbol Connector_Generic:Conn_01x03
- removed J5: 01x08, Connector_PinHeader_2.54mm:PinHeader_1x08_P2.54mm_Vertical, symbol Connector_Generic:Conn_01x08
- removed J6: 01x10, Connector_PinHeader_2.54mm:PinHeader_1x10_P2.54mm_Vertical, symbol Connector_Generic:Conn_01x10
- removed J7: 01x12, Connector_PinHeader_2.54mm:PinHeader_1x12_P2.54mm_Vertical, symbol Connector_Generic:Conn_01x12
- removed SW1: SW4Push, Button_Switch_THT:SW_PUSH_6mm, symbol Switch4Prong:SW4Push
- added J4, J5: Conn_01x17, Connector_PinHeader_2.54mm:PinHeader_1x17_P2.54mm_Vertical, symbol Connector_Generic:Conn_01x17
- added SW1: SW_Push, ExOneFootprints:PTS636SM25SMTRLFS, symbol Switch:SW_Push
Connections:
- net +3.3VA is gone; now on net +3V3: R5.2
- net GND: now also SW1.2
- net PA0: now also J5.1 (Pin_1)
- net PA1: now also J5.17 (Pin_17)
- net PA10: now also J4.16 (Pin_16)
- net PA11: now also J4.15 (Pin_15)
- net PA12: now also J4.14 (Pin_14)
- net PA15: now also J4.13 (Pin_13)
- net PA4: now also J5.3 (Pin_3)
- net PA5: now also J5.4 (Pin_4)
- net PA7: now also J5.5 (Pin_5)
- net PA8: now also J5.14 (Pin_14)
- net PA9: now also J5.15 (Pin_15)
- net PB0: now also J5.6 (Pin_6)
- net PB10: now also J5.8 (Pin_8)
- net PB11: now also J5.9 (Pin_9)
- net PB12: now also J5.10 (Pin_10)
- net PB13: now also J5.11 (Pin_11)
- net PB14: now also J5.12 (Pin_12)
- net PB15: now also J5.13 (Pin_13)
- net PB2: now also J5.7 (Pin_7)
- net PB3: now also J4.8 (Pin_8)
- net PB4: now also J4.7 (Pin_7)
- net PB5: now also J4.6 (Pin_6)
- net PB6: now also J4.5 (Pin_5)
- net PB7: now also J4.4 (Pin_4)
- net PB8: now also J4.3 (Pin_3)
- net PB9: now also J4.2 (Pin_2)
- net PC13: now also J4.1 (Pin_1)
- net PC6: now also J5.16 (Pin_16)
- net PC7: now also J4.17 (Pin_17)
- net PD0: now also J4.12 (Pin_12)
- net PD1: now also J4.11 (Pin_11)
- net PD2: now also J4.10 (Pin_10)
- net PD3: now also J4.9 (Pin_9)
- net at R5.1, R6.1: now also SW1.1
- net VCCIO renamed 3VLn
- no-connect marks 6 -> 7
Changed lines of the file:
@@
 OSC_OUT
-$Comp
-L Switch4Prong:SW4Push SW1
-U 1 1 5E72DBED
-P 1125 3975
-F 0 "SW1" V 1050 3650 50  0000 L CNN
-F 1 "SW4Push" V 1150 3500 50  0000 L CNN
-F 2 "Button_Switch_THT:SW_PUSH_6mm" H 1125 4175 50  0001 C CNN
-F 3 "~" H 1125 4175 50  0001 C CNN
-	1    1125 3975
-	0    1    1    0
-$EndComp
 $Comp
 L Device:R_Small R1
@@
 	1    0    0    -1
 $EndComp
-Wire Wire Line
-	1025 4275 1125 4275
-Connection ~ 1125 4275
-Wire Wire Line
-	1125 4275 1225 4275
 $Comp
 L power:GND #PWR0111
 U 1 1 5E7FECCA
-P 1125 4375
-F 0 "#PWR0111" H 1125 4125 50  0001 C CNN
-F 1 "GND" H 1125 4225 50  0000 C CNN
-F 2 "" H 1125 4375 50  0001 C CNN
-F 3 "" H 1125 4375 50  0001 C CNN
-	1    1125 4375
-	1    0    0    -1
-$EndComp
-Wire Wire Line
-	1125 4275 1125 4375
+P 1125 4075
+F 0 "#PWR0111" H 1125 3825 50  0001 C CNN
+F 1 "GND" H 1125 3925 50  0000 C CNN
+F 2 "" H 1125 4075 50  0001 C CNN
+F 3 "" H 1125 4075 50  0001 C CNN
+	1    1125 4075
+	1    0    0    -1
+$EndComp
 $Comp
 L Connector_Generic:Conn_02x03_Odd_Even J3
@@
 Text GLabel 6950 3825 0    50   Input ~ 0
 RTS
-$Comp
-L Connector_Generic:Conn_01x03 J4
-U 1 1 5E8E29D2
-P 10075 3025
-F 0 "J4" H 10025 3225 50  0000 L CNN
-F 1 "01x03" H 9950 2825 50  0000 L CNN
-F 2 "Connector_PinHeader_2.54mm:PinHeader_1x03_P2.54mm_Vertical" H 10075 3025 50  0001 C CNN
-F 3 "~" H 10075 3025 50  0001 C CNN
-	1    10075 3025
-	1    0    0    -1
-$EndComp
-$Comp
-L Connector_Generic:Conn_01x08 J5
-U 1 1 5E8E2FAE
-P 10075 4000
-F 0 "J5" H 10025 4400 50  0000 L CNN
-F 1 "01x08" H 9950 3500 50  0000 L CNN
-F 2 "Connector_PinHeader_2.54mm:PinHeader_1x08_P2.54mm_Vertical" H 10075 4000 50  0001 C CNN
-F 3 "~" H 10075 4000 50  0001 C CNN
-	1    10075 4000
-	1    0    0    -1
-$EndComp
-$Comp
-L Connector_Generic:Conn_01x10 J6
-U 1 1 5E8E69B2
-P 11000 2875
-F 0 "J6" H 10950 3375 50  0000 L CNN
-F 1 "01x10" H 10875 2250 50  0000 L CNN
-F 2 "Connector_PinHeader_2.54mm:PinHeader_1x10_P2.54mm_Vertical" H 11000 2875 50  0001 C CNN
-F 3 "~" H 11000 2875 50  0001 C CNN
-	1    11000 2875
-	1    0    0    -1
-$EndComp
-$Comp
-L Connector_Generic:Conn_01x12 J7
-U 1 1 5E8E732E
-P 11000 4325
-F 0 "J7" H 10950 4925 50  0000 L CNN
-F 1 "01x12" H 10875 3625 50  0000 L CNN
-F 2 "Connector_PinHeader_2.54mm:PinHeader_1x12_P2.54mm_Vertical" H 11000 4325 50  0001 C CNN
-F 3 "~" H 11000 4325 50  0001 C CNN
-	1    11000 4325
-	1    0    0    -1
-$EndComp
-Text GLabel 9875 2925 0    50   BiDi ~ 0
+Text GLabel 9525 2925 0    50   BiDi ~ 0
 PC13
-Text GLabel 9875 3025 0    50   BiDi ~ 0
+Text GLabel 10550 2925 0    50   BiDi ~ 0
 PA0
-Text GLabel 9875 3125 0    50   BiDi ~ 0
+Text GLabel 10550 4525 0    50   BiDi ~ 0
 PA1
 Text GLabel 6950 2625 0    50   BiDi ~ 0
@@
 Text GLabel 6950 3325 0    50   BiDi ~ 0
 PA1
-Text GLabel 9875 3700 0    50   BiDi ~ 0
+Text GLabel 10550 3125 0    50   BiDi ~ 0
 PA4
 Text GLabel 6950 3625 0    50   BiDi ~ 0
 PA4
-Text GLabel 9875 3800 0    50   BiDi ~ 0
+Text GLabel 10550 3225 0    50   BiDi ~ 0
 PA5
 Text GLabel 6950 3725 0    50   BiDi ~ 0
 PA5
-Text GLabel 9875 3900 0    50   BiDi ~ 0
+Text GLabel 10550 3325 0    50   BiDi ~ 0
 PA7
 Text GLabel 6950 3925 0    50   BiDi ~ 0
 PA7
-Text GLabel 9875 4000 0    50   BiDi ~ 0
+Text GLabel 10550 3425 0    50   BiDi ~ 0
 PB0
 Text GLabel 6950 4025 0    50   BiDi ~ 0
 PB0
-Text GLabel 9875 4100 0    50   BiDi ~ 0
+Text GLabel 10550 3525 0    50   BiDi ~ 0
 PB2
 Text GLabel 6950 4225 0    50   BiDi ~ 0
 PB2
-Text GLabel 9875 4200 0    50   BiDi ~ 0
+Text GLabel 10550 3625 0    50   BiDi ~ 0
 PB10
 Text GLabel 6950 4325 0    50   BiDi ~ 0
 PB10
-Text GLabel 9875 4300 0    50   BiDi ~ 0
+Text GLabel 10550 3725 0    50   BiDi ~ 0
 PB11
 Text GLabel 6950 4425 0    50   BiDi ~ 0
 PB11
-Text GLabel 9875 4400 0    50   BiDi ~ 0
+Text GLabel 10550 3825 0    50   BiDi ~ 0
 PB12
 Text GLabel 6950 4525 0    50   BiDi ~ 0
@@
 Text GLabel 8700 2825 2    50   BiDi ~ 0
 PA12
-Text GLabel 10800 2475 0    50   BiDi ~ 0
+Text GLabel 9525 4225 0    50   BiDi ~ 0
 PA12
 Text GLabel 8700 2925 2    50   BiDi ~ 0
 PA11
-Text GLabel 10800 2575 0    50   BiDi ~ 0
+Text GLabel 9525 4325 0    50   BiDi ~ 0
 PA11
-Text GLabel 10800 2675 0    50   BiDi ~ 0
+Text GLabel 9525 4425 0    50   BiDi ~ 0
 PA10
 Text GLabel 8700 3025 2    50   BiDi ~ 0
 PA10
-Text GLabel 10800 2775 0    50   BiDi ~ 0
+Text GLabel 9525 4525 0    50   BiDi ~ 0
 PC7
 Text GLabel 8700 3125 2    50   BiDi ~ 0
 PC7
-Text GLabel 10800 2875 0    50   BiDi ~ 0
+Text GLabel 10550 4425 0    50   BiDi ~ 0
 PC6
 Text GLabel 8700 3225 2    50   BiDi ~ 0
 PC6
-Text GLabel 10800 2975 0    50   BiDi ~ 0
+Text GLabel 10550 4325 0    50   BiDi ~ 0
 PA9
 Text GLabel 8700 3325 2    50   BiDi ~ 0
 PA9
-Text GLabel 10800 3075 0    50   BiDi ~ 0
+Text GLabel 10550 4225 0    50   BiDi ~ 0
 PA8
 Text GLabel 8700 3425 2    50   BiDi ~ 0
 PA8
-Text GLabel 10800 3175 0    50   BiDi ~ 0
+Text GLabel 10550 4125 0    50   BiDi ~ 0
 PB15
 Text GLabel 8700 3525 2    50   BiDi ~ 0
 PB15
-Text GLabel 10800 3275 0    50   BiDi ~ 0
+Text GLabel 10550 4025 0    50   BiDi ~ 0
 PB14
 Text GLabel 8700 3625 2    50   BiDi ~ 0
 PB14
-Text GLabel 10800 3375 0    50   BiDi ~ 0
+Text GLabel 10550 3925 0    50   BiDi ~ 0
 PB13
 Text GLabel 8700 3725 2    50   BiDi ~ 0
 PB13
-Text GLabel 10800 3825 0    50   BiDi ~ 0
+Text GLabel 9525 3025 0    50   BiDi ~ 0
 PB9
-Text GLabel 10800 3925 0    50   BiDi ~ 0
+Text GLabel 9525 3125 0    50   BiDi ~ 0
 PB8
 Text GLabel 8700 3825 2    50   BiDi ~ 0
@@
 Text GLabel 8700 3925 2    50   BiDi ~ 0
 PB8
-Text GLabel 10800 4025 0    50   BiDi ~ 0
+Text GLabel 9525 3225 0    50   BiDi ~ 0
 PB7
 Text GLabel 8700 4025 2    50   BiDi ~ 0
 PB7
-Text GLabel 10800 4125 0    50   BiDi ~ 0
+Text GLabel 9525 3325 0    50   BiDi ~ 0
 PB6
 Text GLabel 8700 4125 2    50   BiDi ~ 0
 PB6
-Text GLabel 10800 4225 0    50   BiDi ~ 0
+Text GLabel 9525 3425 0    50   BiDi ~ 0
 PB5
 Text GLabel 8700 4225 2    50   BiDi ~ 0
 PB5
-Text GLabel 10800 4325 0    50   BiDi ~ 0
+Text GLabel 9525 3525 0    50   BiDi ~ 0
 PB4
 Text GLabel 8700 4325 2    50   BiDi ~ 0
 PB4
-Text GLabel 10800 4425 0    50   BiDi ~ 0
+Text GLabel 9525 3625 0    50   BiDi ~ 0
 PB3
 Text GLabel 8700 4425 2    50   BiDi ~ 0
 PB3
-Text GLabel 10800 4525 0    50   BiDi ~ 0
+Text GLabel 9525 3725 0    50   BiDi ~ 0
 PD3
 Text GLabel 8700 4525 2    50   BiDi ~ 0
@@
 Text GLabel 8700 4625 2    50   BiDi ~ 0
 PD2
-Text GLabel 10800 4625 0    50   BiDi ~ 0
+Text GLabel 9525 3825 0    50   BiDi ~ 0
 PD2
 Text GLabel 8700 4725 2    50   BiDi ~ 0
 PD1
-Text GLabel 10800 4725 0    50   BiDi ~ 0
+Text GLabel 9525 3925 0    50   BiDi ~ 0
 PD1
-Text GLabel 10800 4825 0    50   BiDi ~ 0
+Text GLabel 9525 4025 0    50   BiDi ~ 0
 PD0
 Text GLabel 8700 4825 2    50   BiDi ~ 0
@@
 Text GLabel 8700 4925 2    50   BiDi ~ 0
 PA15
-Text GLabel 10800 4925 0    50   BiDi ~ 0
+Text GLabel 9525 4125 0    50   BiDi ~ 0
 PA15
 Wire Notes Line
@@
 	4350 3225 4825 3225
 Wire Wire Line
-	1025 3675 1125 3675
-Wire Wire Line
 	1125 3675 1125 3600
 Connection ~ 1125 3675
-Wire Wire Line
-	1125 3675 1225 3675
 $Comp
 L Device:R_Small R5
@@
 	1125 3400 1125 3300
 $Comp
-L power:+3.3VA #PWR0122
-U 1 1 5EBBC3C0
-P 1125 3300
-F 0 "#PWR0122" H 1125 3150 50  0001 C CNN
-F 1 "+3.3VA" H 950 3350 50  0000 C CNN
-F 2 "" H 1125 3300 50  0001 C CNN
-F 3 "" H 1125 3300 50  0001 C CNN
-	1    1125 3300
-	1    0    0    -1
-$EndComp
-$Comp
 L Device:R_Small R6
 U 1 1 5EBCCA59
@@
 	0    -1   -1   0
 $EndComp
-Wire Wire Line
-	1500 3675 1225 3675
-Connection ~ 1225 3675
 $Comp
 L Device:C C14
@@
 	4175 6350 4175 6850
 Text GLabel 4075 5450 0    50   Output ~ 0
-VCCIO
+3VLn
 Text GLabel 4075 6350 0    50   Input ~ 0
-VCCIO
+3VLn
 Wire Wire Line
 	4175 6350 4075 6350
@@
 Wire Wire Line
 	4075 5450 4225 5450
+$Comp
+L power:+3V3 #PWR0116
+U 1 1 5E7DB2B1
+P 1125 3300
+F 0 "#PWR0116" H 1125 3150 50  0001 C CNN
+F 1 "+3V3" H 1150 3525 50  0000 C CNN
+F 2 "" H 1125 3300 50  0001 C CNN
+F 3 "" H 1125 3300 50  0001 C CNN
+	1    1125 3300
+	1    0    0    -1
+$EndComp
+$Comp
+L Connector_Generic:Conn_01x17 J4
+U 1 1 5E7F012C
+P 9725 3725
+F 0 "J4" H 9675 4650 50  0000 L CNN
+F 1 "Conn_01x17" H 9325 2775 50  0000 L CNN
+F 2 "Connector_PinHeader_2.54mm:PinHeader_1x17_P2.54mm_Vertical" H 9725 3725 50  0001 C CNN
+F 3 "~" H 9725 3725 50  0001 C CNN
+	1    9725 3725
+	1    0    0    -1
+$EndComp
+$Comp
+L Connector_Generic:Conn_01x17 J5
+U 1 1 5E7F19A5
+P 10750 3725
+F 0 "J5" H 10700 4650 50  0000 L CNN
+F 1 "Conn_01x17" H 10350 2775 50  0000 L CNN
+F 2 "Connector_PinHeader_2.54mm:PinHeader_1x17_P2.54mm_Vertical" H 10750 3725 50  0001 C CNN
+F 3 "~" H 10750 3725 50  0001 C CNN
+	1    10750 3725
+	1    0    0    -1
+$EndComp
+NoConn ~ 10550 3025
+$Comp
+L Switch:SW_Push SW1
+U 1 1 5E90B04D
+P 1125 3875
+F 0 "SW1" V 1050 4050 50  0000 L CNN
+F 1 "SW_Push" V 1150 4050 50  0000 L CNN
+F 2 "ExOneFootprints:PTS636SM25SMTRLFS" H 1125 4075 50  0001 C CNN
+F 3 "~" H 1125 4075 50  0001 C CNN
+	1    1125 3875
+	0    1    1    0
+$EndComp
+Wire Wire Line
+	1125 3675 1500 3675
 $EndSCHEMATC

Commit message: FInished work on pcb , added some pads for 3v3 and gnd
Parts:
- added J6: Conn_01x02, Connector_PinHeader_2.54mm:PinHeader_1x02_P2.54mm_Vertical, symbol Connector_Generic:Conn_01x02
Connections:
- net +3V3: now also J6.1 (Pin_1)
- net GND: now also J5.2 (Pin_2), J6.2 (Pin_2)
- no-connect marks 7 -> 6
Changed lines of the file:
@@
 $EndComp
-$Comp
-L Connector_Generic:Conn_01x17 J5
-U 1 1 5E7F19A5
-P 10750 3725
-F 0 "J5" H 10700 4650 50  0000 L CNN
-F 1 "Conn_01x17" H 10350 2775 50  0000 L CNN
-F 2 "Connector_PinHeader_2.54mm:PinHeader_1x17_P2.54mm_Vertical" H 10750 3725 50  0001 C CNN
-F 3 "~" H 10750 3725 50  0001 C CNN
-	1    10750 3725
-	1    0    0    -1
-$EndComp
-NoConn ~ 10550 3025
 $Comp
 L Switch:SW_Push SW1
@@
 Wire Wire Line
 	1125 3675 1500 3675
+$Comp
+L Connector_Generic:Conn_01x02 J6
+U 1 1 5E79CAF4
+P 10125 5575
+F 0 "J6" H 10250 5600 50  0000 L CNN
+F 1 "Conn_01x02" H 10250 5500 50  0000 L CNN
+F 2 "Connector_PinHeader_2.54mm:PinHeader_1x02_P2.54mm_Vertical" H 10125 5575 50  0001 C CNN
+F 3 "~" H 10125 5575 50  0001 C CNN
+	1    10125 5575
+	1    0    0    -1
+$EndComp
+$Comp
+L Connector_Generic:Conn_01x17 J5
+U 1 1 5E7F19A5
+P 10750 3725
+F 0 "J5" H 10700 4650 50  0000 L CNN
+F 1 "Conn_01x17" H 10350 2775 50  0000 L CNN
+F 2 "Connector_PinHeader_2.54mm:PinHeader_1x17_P2.54mm_Vertical" H 10750 3725 50  0001 C CNN
+F 3 "~" H 10750 3725 50  0001 C CNN
+	1    10750 3725
+	1    0    0    -1
+$EndComp
+Wire Wire Line
+	10200 3025 10550 3025
+$Comp
+L power:GND #PWR0117
+U 1 1 5E7A3E95
+P 10200 3025
+F 0 "#PWR0117" H 10200 2775 50  0001 C CNN
+F 1 "GND" H 10250 2800 50  0000 C CNN
+F 2 "" H 10200 3025 50  0001 C CNN
+F 3 "" H 10200 3025 50  0001 C CNN
+	1    10200 3025
+	1    0    0    -1
+$EndComp
+$Comp
+L power:+3V3 #PWR0122
+U 1 1 5E7A63F6
+P 9925 5575
+F 0 "#PWR0122" H 9925 5425 50  0001 C CNN
+F 1 "+3V3" H 9950 5800 50  0000 C CNN
+F 2 "" H 9925 5575 50  0001 C CNN
+F 3 "" H 9925 5575 50  0001 C CNN
+	1    9925 5575
+	1    0    0    -1
+$EndComp
+$Comp
+L power:GND #PWR0133
+U 1 1 5E7A6886
+P 9925 5675
+F 0 "#PWR0133" H 9925 5425 50  0001 C CNN
+F 1 "GND" H 9950 5450 50  0000 C CNN
+F 2 "" H 9925 5675 50  0001 C CNN
+F 3 "" H 9925 5675 50  0001 C CNN
+	1    9925 5675
+	1    0    0    -1
+$EndComp
 $EndSCHEMATC

Commit message: made prod files JLC complimant
Parts:
- C1, C14, C15, C18: LCSC (none) -> C19666
- IC1: LCSC (none) -> C432202
- IC2: LCSC (none) -> C69082
- U1: LCSC (none) -> C202171
Changed lines of the file:
@@
 EESchema Schematic File Version 4
-LIBS:ExOneMicrorocessor-cache
 EELAYER 30 0
 EELAYER END
@@
 F 2 "ExOneFootprints:FT230XS" H 5025 6500 50  0001 L BNN
 F 3 "" H 4925 5950 50  0001 C CNN
+F 4 "C69082" H 4925 5950 50  0001 C CNN "LCSC"
 	1    4925 5950
 	1    0    0    -1
@@
 F 2 "Capacitor_SMD:C_0603_1608Metric_Pad1.05x0.95mm_HandSolder" H 4963 1375 50  0001 C CNN
 F 3 "~" H 4925 1525 50  0001 C CNN
+F 4 "C19666" H 4925 1525 50  0001 C CNN "LCSC"
 	1    4925 1525
 	-1   0    0    1
@@
 F 8 "STMicroelectronics" H 9200 4125 50  0001 L CNN "Manufacturer_Name"
 F 9 "STM32G041C8T6" H 9200 4025 50  0001 L CNN "Manufacturer_Part_Number"
+F 10 "C432202" H 6950 3625 50  0001 C CNN "LCSC"
 	1    6950 3625
 	1    0    0    -1
@@
 F 2 "Capacitor_SMD:C_0603_1608Metric_Pad1.05x0.95mm_HandSolder" H 2163 3675 50  0001 C CNN
 F 3 "~" H 2125 3825 50  0001 C CNN
+F 4 "C19666" H 2125 3825 50  0001 C CNN "LCSC"
 	1    2125 3825
 	-1   0    0    1
@@
 F 6 "SOIC-8" H 4825 1275 50  0001 L BNN "Field6"
 F 7 "Texas Instruments" H 4675 1525 50  0001 L BNN "Field7"
+F 8 "C202171" H 3575 1375 50  0001 C CNN "LCSC"
 	1    3575 1375
 	1    0    0    -1
@@
 F 2 "Capacitor_SMD:C_0603_1608Metric_Pad1.05x0.95mm_HandSolder" H 6288 5600 50  0001 C CNN
 F 3 "~" H 6250 5750 50  0001 C CNN
+F 4 "C19666" H 6250 5750 50  0001 C CNN "LCSC"
 	1    6250 5750
 	-1   0    0    1
@@
 F 2 "Capacitor_SMD:C_0603_1608Metric_Pad1.05x0.95mm_HandSolder" H 8763 925 50  0001 C CNN
 F 3 "~" H 8725 1075 50  0001 C CNN
+F 4 "C19666" H 8725 1075 50  0001 C CNN "LCSC"
 	1    8725 1075
 	-1   0    0    1
